Commit message: fixed collision

File: src/lab2andDriver/drivers/universal_robot/ur_description/urdf/ur3.urdf.xacro (robot description, xacro)
@@ -314,5 +314,5 @@
       <collision>
         <geometry>
-          <box size="0.01 0.01 0.01"/>
+          <box size="0.048 0.101 0.04"/>
         </geometry>
         <surface>
@@ -324,5 +324,5 @@
           </friction>
         </surface>
-        <origin rpy="0 0 0" xyz="-0.01 0 0"/>
+        <origin rpy="0 0 0" xyz="0.023 0.02 0.0"/>
       </collision>
       <inertial>
